File: Hardware/9DoF_Sensor_Stick.brd (EAGLE design)
At the start: 34.3 x 10.2 mm, 31 parts, among them U1 ITG-3200, U2 ADXL345, U4 3.3V

Commit message: comp change
Parts:
- moved R5 23.2 mm to (16.8, 8.02), turned to 90 degrees
- moved U$5 20.0 mm to (15.9, 4.62), turned to 270 degrees
- moved R4 11.9 mm to (15.1, 1.07)
- moved U$4 9.38 mm to (13.7, 4.61), turned to 90 degrees
- moved C5 7.09 mm to (23.6, 8.91)
- moved C6 6.02 mm to (32.6, 1.28), turned to 180 degrees
- moved C1 5.85 mm to (18.3, 8.01)
- moved C4 5.25 mm to (19.4, 1.11)
- moved C3 5.24 mm to (19.4, 2.45)
- moved R3 4.84 mm to (25.7, 1.28)
- moved LED1 4.81 mm to (22.6, 1.26)
- moved R1 4.64 mm to (11.0, 1.07)
- moved C8 4.39 mm to (28.5, 8.89)
- moved U1 4.39 mm to (28.5, 5.08)
- moved C7 4.29 mm to (24.6, 5.53)
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Routing:
- net SCL: track 41.4 -> 61.8 mm
- net 3.3V: track 43.7 -> 58.3 mm
- net GND: track 32.7 -> 41.7 mm
- net N$3: track 12.1 -> 4.65 mm, vias 2 -> 1
- net N$8: track 0.00 -> 4.89 mm
- net SDA: track 37.4 -> 42.0 mm
- net N$5: track 1.85 -> 4.67 mm
- net N$9: track 0.00 -> 2.14 mm
- net N$2: track 5.64 -> 4.08 mm
- net N$1: track 2.17 -> 1.43 mm
Other:
- board size 34.3 x 10.2 mm -> 36.8 x 10.2 mm

Commit message: comp change
Parts:
- removed JP4: LOGO-SFESK, SparkFun:SFE-LOGO-FLAME
- removed U$1: CREATIVE_COMMONS, SparkFun:CREATIVE_COMMONS
- added FRAME1: FRAME-LETTER, SparkFun-Aesthetics:CREATIVE_COMMONS
- moved R2 2.15 mm to (5.04, 8.87)
- moved C10 2.06 mm to (8.66, 8.90)
- moved C5 1.26 mm to (22.4, 8.58)
- moved C1 1.25 mm to (17.1, 7.71)
- moved R5 1.22 mm to (15.6, 7.70), turned to 270 degrees
- moved C2 1.00 mm to (14.1, 7.72), turned to 90 degrees
- moved U$5 0.88 mm to (16.6, 4.03)
- moved U$4 0.62 mm to (13.9, 4.01)
- moved C6 0.47 mm to (32.6, 0.82)
- moved LED1 0.47 mm to (22.5, 0.80)
- moved R3 0.47 mm to (25.7, 0.81)
- moved C9 0.47 mm to (29.1, 0.81)
- moved C4 0.26 mm to (19.4, 0.85)
- moved C3 0.24 mm to (19.4, 2.21)
- moved R4 0.24 mm to (15.2, 0.83)
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Connections:
- net N$10: now also U$5.2
Routing:
- net GND: track 41.7 -> 5.15 mm, vias 4 -> 1
- net SCL: track 61.8 -> 51.3 mm
- net 3.3V: track 58.3 -> 50.9 mm
- net N$6: track 0.00 -> 4.65 mm
- net N$9: track 2.14 -> 4.10 mm
- net N$8: track 4.89 -> 3.66 mm
Other:
- board text added: "Revised by: Patrick Alberts"
